File: SC_LED_CUBE_SLAVE_Board/SC_LED_CUBE_SLAVE_Board.kicad_pcb (KiCad board)
At the start: 2 copper layers, 98 x 98 mm, 127 parts, among them CN1 XT30UPB-M, CN2 B03B-XASK-1-A(LF)(SN), CN3 B03B-XASK-1-A(LF)(SN), CN4 B03B-XASK-1-A(LF)(SN), CN5 B03B-XASK-1-A(LF)(SN), Q1 SIL2305B-TP, Q10 SIL2305B-TP, Q11 SIL2305B-TP, Q12 SIL2305B-TP, Q2 PMZ600UNEYL, Q3 PMZ600UNEYL, Q4 SIL2305B-TP, Q5 SIL2305B-TP, Q6 SIL2305B-TP, Q7 SIL2305B-TP, Q8 SIL2305B-TP, Q9 SIL2305B-TP, U1 SN74LVC1G14DBV, U10 SN74LVC1G14DBV, U11 SN74LVC1G14DBV, U12 SN74LVC1G14DBV, U13 SN74LVC1G14DBV, U14 SN74LVC1G14DBV, U15 74AHC164S14-13, U2 STP16CPC26XTR, U3 STP16CPC26XTR, U5 74AHC164S14-13, U6 SN74LVC1G14DBV, U7 SN74LVC1G14DBV, U8 SN74LVC1G14DBV, U9 SN74LVC1G14DBV

Commit message: Finished the layout 0 DRC errors.
Parts:
- added C44: 100uF, Capacitor_SMD:C_1206_3216Metric_Pad1.33x1.80mm_HandSolder, B.Cu at (117.8, 70.0)
- added C45: 100uF, Capacitor_SMD:C_1206_3216Metric_Pad1.33x1.80mm_HandSolder, B.Cu at (139.2, 70.4)
- added C46: 100uF, Capacitor_SMD:C_1206_3216Metric_Pad1.33x1.80mm_HandSolder, B.Cu at (164.3, 72.5)
- added C47: 100uF, Capacitor_SMD:C_1206_3216Metric_Pad1.33x1.80mm_HandSolder, B.Cu at (177.9, 70.1)
- added C48: 100uF, Capacitor_SMD:C_1206_3216Metric_Pad1.33x1.80mm_HandSolder, B.Cu at (104.5, 73.2)
- added C49: 270uF, Capacitor_THT:CP_Radial_D6.3mm_P2.50mm, F.Cu at (180.0, 141.5)
- added R46: 0R, Resistor_SMD:R_0402_1005Metric_Pad0.72x0.64mm_HandSolder, F.Cu at (158.4, 93.2)
- added R47: 0R, Resistor_SMD:R_0402_1005Metric_Pad0.72x0.64mm_HandSolder, F.Cu at (126.4, 106.1)
- moved Q12 445.4 mm to (180.6, 59.7), turned to -90 degrees
- moved C34 436.0 mm to (181.8, 62.6), turned to -90 degrees
- moved R15 430.2 mm to (179.4, 62.9)
- moved Q9 427.9 mm to (120.6, 59.7), turned to -90 degrees
- moved C33 421.6 mm to (183.6, 62.9), turned to -90 degrees
- moved C29 418.6 mm to (121.8, 62.6), turned to -90 degrees
- moved C32 412.7 mm to (180.3, 68.7)
- moved R12 412.7 mm to (119.5, 62.9)
- moved Q10 409.9 mm to (140.6, 59.7), turned to -90 degrees
- moved U14 408.9 mm to (180.6, 66.3), turned to 180 degrees
- moved C26 404.2 mm to (123.6, 62.9), turned to -90 degrees
- moved Q11 400.0 mm to (160.6, 59.7), turned to -90 degrees
- moved C30 398.5 mm to (141.8, 62.6), turned to -90 degrees
- moved C23 395.3 mm to (120.3, 68.7)
- moved R13 394.3 mm to (139.4, 62.9)
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Connections:
- R1 pad 1: Net-(U2-R-EXT) -> Net-(R1-Pad1)
- R6 pad 1: /R_EXT -> Net-(R47-Pad1)
Routing:
- net Net-(Q2-G): track 0.00 -> 107.0 mm, vias 0 -> 6
- net /OE: track 0.00 -> 69.2 mm, vias 0 -> 6
- net /O20: track 0.00 -> 68.6 mm, vias 0 -> 8
- net /Layer_Switching/Q4: track 0.00 -> 67.8 mm, vias 0 -> 6
- net /LE: track 0.00 -> 55.9 mm, vias 0 -> 4
- net /O24: track 0.00 -> 55.4 mm, vias 0 -> 4
- net /O19: track 0.00 -> 55.3 mm, vias 0 -> 4
- net /CLK: track 0.00 -> 54.2 mm, vias 0 -> 4
- net /Layer_Switching/Q5: track 0.00 -> 52.6 mm, vias 0 -> 4
- net /O23: track 0.00 -> 51.8 mm
- net /O21: track 0.00 -> 50.4 mm, vias 0 -> 4
- net /Layer_Switching/Q0: track 0.00 -> 48.0 mm, vias 0 -> 2
- net /Layer_Switching/Q3: track 0.00 -> 47.7 mm, vias 0 -> 4
- net /O15: track 0.00 -> 41.5 mm
- net /O10: track 0.00 -> 39.9 mm, vias 0 -> 4
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- added copper zone on B.Cu, net +3V3
- added copper zone on F.Cu, net +3V3
- added copper zone on B.Cu, net /Layer_Switching/L0
- added copper zone on F.Cu, net /Layer_Switching/L0
- added copper zone on B.Cu, net /Layer_Switching/L1
- added copper zone on F.Cu, net /Layer_Switching/L1
- added copper zone on B.Cu, net /Layer_Switching/L2
- added copper zone on F.Cu, net /Layer_Switching/L2
- added copper zone on B.Cu, net /Layer_Switching/L3
- added copper zone on F.Cu, net /Layer_Switching/L3
- added copper zone on B.Cu, net /Layer_Switching/L4
- added copper zone on F.Cu, net /Layer_Switching/L4
- added copper zone on B.Cu, net /Layer_Switching/L5
- added copper zone on F.Cu, net /Layer_Switching/L5
- added copper zone on B.Cu, net /Layer_Switching/L6
- added copper zone on F.Cu, net /Layer_Switching/L6
- added copper zone on B.Cu, net /Layer_Switching/L7
- added copper zone on F.Cu, net /Layer_Switching/L7
- added copper zone on B.Cu, net /Layer_Switching/L8
- added copper zone on F.Cu, net /Layer_Switching/L8
- added copper zone on B.Cu, net /Layer_Switching/L9
- added copper zone on F.Cu, net /Layer_Switching/L9
- added copper zone on B.Cu, net GND
- added copper zone on F.Cu, net GND
- added copper zone on B.Cu, net VCC
- added copper zone on F.Cu, net VCC

Commit message: Small mostly cosmetic changes, followed by the export of the gerber files for production.
Parts:
- added G***: LOGO, LOGO, F.Cu at (161.5, 146.7)
- added G***: LOGO, LOGO, F.Cu at (123.8, 134.5)
- added G***: LOGO, LOGO, F.Cu at (180.9, 89.4)
- added G***: LOGO, LOGO, F.Cu at (113.1, 137.4)
- added G***: LOGO, LOGO, F.Cu at (119.1, 131.4)
- added REF**: OSHW-Logo2_14.6x12mm_SilkScreen, Symbol:OSHW-Logo2_14.6x12mm_SilkScreen, F.Cu at (135.8, 142.0)
- added REF**: ESD-Logo_13.2x12mm_SilkScreen, Symbol:ESD-Logo_13.2x12mm_SilkScreen, F.Cu at (135.2, 128.2)
- added kobee-studio-6AA92370: Kobee Studio, kobee-studio-6AA92370, F.Cu at (118.1, 146.6)
- added kobee-studio-6AA93567: Kobee Studio, kobee-studio-6AA93567, F.Cu at (147.2, 146.7)
- added kobee-studio-6AA935D6: Kobee Studio, kobee-studio-6AA935D6, F.Cu at (115.8, 117.4)
- added kobee-studio-6AA936F7: Kobee Studio, kobee-studio-6AA9368C, F.Cu at (145.4, 130.4)
- moved CN3 17.5 mm to (183.1, 130.4)
- moved CN2 15.0 mm to (165.1, 130.4)
- moved CN1 2.58 mm to (156.1, 130.4)
- moved CN4 1.10 mm to (174.1, 130.4)
- renumbered C3 to C1, C42 to C10, C41 to C11, C40 to C12, C39 to C13, C38 to C14, C43 to C15, C49 to C16, C32 to C17, C33 to C18, C34 to C19, C1 to C2, C23 to C20, C26 to C21, C29 to C22, C14 to C23, C17 to C24, C20 to C25, C6 to C26, C5 to C27, C7 to C28, C24 to C29, C4 to C3, C27 to C30, C30 to C31, C15 to C32, C18 to C33, C21 to C34, C8 to C35, C9 to C36, C10 to C37, C25 to C38, C28 to C39, C2 to C4, C31 to C40, C16 to C41, C19 to C42, C22 to C43, C11 to C44, C12 to C45, C13 to C46, C35 to C47, C36 to C48, C37 to C49, C48 to C5, C44 to C6, C45 to C7, C46 to C8, C47 to C9, CN4 to CN1, CN5 to CN3, CN3 to CN4, CN1 to CN5, FPC2 to FPC1, FPC1 to FPC2, Q2 to Q1, Q11 to Q10, Q8 to Q11, Q5 to Q12, Q3 to Q2, Q12 to Q3, Q9 to Q4, Q6 to Q5, Q1 to Q6, Q10 to Q7, Q7 to Q8, Q4 to Q9, R21 to R1, R26 to R10, R27 to R11, R28 to R12, R29 to R13, R30 to R14, R20 to R15, R2 to R16, R7 to R17, R5 to R18, R31 to R19, R22 to R2, R32 to R20, R33 to R21, R34 to R22, R35 to R23, R36 to R24, R37 to R25, R38 to R26, R39 to R27, R40 to R28, R16 to R29, R23 to R3, R41 to R30, R42 to R31, R43 to R32, R44 to R33, R45 to R34, R15 to R35, R12 to R36, R9 to R37, R3 to R38, R13 to R39, R24 to R4, R10 to R40, R4 to R41, R14 to R42, R11 to R43, R8 to R44, R17 to R45, R18 to R46, R19 to R47, R25 to R5, R46 to R6, R47 to R7, R1 to R8, R6 to R9, U3 to U1, U13 to U10, U10 to U11, U7 to U12, U5 to U13, U15 to U14, U14 to U3, U11 to U4, U8 to U5, U1 to U6, U12 to U7, U9 to U8, U6 to U9
Routing:
- net /O4: track 59.6 -> 62.7 mm
- net /O3: track 40.6 -> 43.3 mm
- net /O19: track 55.3 -> 57.3 mm
- net /O2: track 26.9 -> 27.5 mm
- net VCC: vias 533 -> 532
- net GND: vias 830 -> 815
Other:
- board text added: "-- . - ..- .-.."
