File: SC_LED_CUBE_SLAVE_Board/SC_LED_CUBE_SLAVE_Board.kicad_pcb (KiCad board)
At the start: 2 copper layers, 98 x 98 mm, 146 parts, among them CN1 B03B-XASK-1-A(LF)(SN), CN2 B03B-XASK-1-A(LF)(SN), CN3 B03B-XASK-1-A(LF)(SN), CN4 B03B-XASK-1-A(LF)(SN), CN5 XT30UPB-M, Q1 PMZ600UNEYL, Q10 SIL2305B-TP, Q11 SIL2305B-TP, Q12 SIL2305B-TP, Q2 PMZ600UNEYL, Q3 SIL2305B-TP, Q4 SIL2305B-TP, Q5 SIL2305B-TP, Q6 SIL2305B-TP, Q7 SIL2305B-TP, Q8 SIL2305B-TP, Q9 SIL2305B-TP, U1 STP16CPC26XTR, U10 SN74LVC1G14DBV, U11 SN74LVC1G14DBV, U12 SN74LVC1G14DBV, U13 74AHC164S14-13, U14 74AHC164S14-13, U2 STP16CPC26XTR, U3 SN74LVC1G14DBV, U4 SN74LVC1G14DBV, U5 SN74LVC1G14DBV, U6 SN74LVC1G14DBV, U7 SN74LVC1G14DBV, U8 SN74LVC1G14DBV, U9 SN74LVC1G14DBV

Commit message: Created design variants changed two components values and added interactive HTML BOM via plugin.
Parts:
- R35, R36, R37, R38, R39, R40, R41, R42, R43, R44: value 10R -> 100R
