File: SC_LED_CUBE_SLAVE_Board/Layer_Switching.kicad_sch (KiCad schematic)
At the start: 68 parts, among them Q1 SIL2305B-TP, Q10 SIL2305B-TP, Q11 SIL2305B-TP, Q12 SIL2305B-TP, Q4 SIL2305B-TP, Q5 SIL2305B-TP, Q6 SIL2305B-TP, Q7 SIL2305B-TP, Q8 SIL2305B-TP, Q9 SIL2305B-TP, U1 SN74LVC1G14DBV, U10 SN74LVC1G14DBV, U11 SN74LVC1G14DBV, U12 SN74LVC1G14DBV, U13 SN74LVC1G14DBV, U14 SN74LVC1G14DBV, U15 74AHC164S14-13, U5 74AHC164S14-13, U6 SN74LVC1G14DBV, U7 SN74LVC1G14DBV, U8 SN74LVC1G14DBV, U9 SN74LVC1G14DBV

Commit message: Small mostly cosmetic changes, followed by the export of the gerber files for production.
Parts:
- renumbered C32 to C17, C33 to C18, C34 to C19, C23 to C20, C26 to C21, C29 to C22, C14 to C23, C17 to C24, C20 to C25, C6 to C26, C5 to C27, C7 to C28, C24 to C29, C27 to C30, C30 to C31, C15 to C32, C18 to C33, C21 to C34, C8 to C35, C9 to C36, C10 to C37, C25 to C38, C28 to C39, C31 to C40, C16 to C41, C19 to C42, C22 to C43, C11 to C44, C12 to C45, C13 to C46, C35 to C47, C36 to C48, C37 to C49, Q11 to Q10, Q8 to Q11, Q5 to Q12, Q12 to Q3, Q9 to Q4, Q6 to Q5, Q1 to Q6, Q10 to Q7, Q7 to Q8, Q4 to Q9, R15 to R35, R12 to R36, R9 to R37, R3 to R38, R13 to R39, R10 to R40, R4 to R41, R14 to R42, R11 to R43, R8 to R44, R17 to R45, R18 to R46, R19 to R47, U13 to U10, U10 to U11, U7 to U12, U5 to U13, U15 to U14, U14 to U3, U11 to U4, U8 to U5, U1 to U6, U12 to U7, U9 to U8, U6 to U9

Commit message: Created design variants changed two components values and added interactive HTML BOM via plugin.
Parts:
- R35, R36, R37, R38, R39, R40, R41, R42, R43, R44: value 10R -> 100R
Changed lines of the file:
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@@
 			)
 		)
-		(property "Value" "10R"
+		(property "Value" "100R"
 			(at 224.79 106.045 90)
 			(show_name no)
@@
 					(reference "R39")
 					(unit 1)
+					(variant
+						(name "5x5x5")
+						(dnp yes)
+					)
 				)
 			)
@@
 					(reference "U11")
 					(unit 1)
+					(variant
+						(name "5x5x5")
+						(dnp yes)
+					)
 				)
 			)
@@
 					(reference "Q4")
 					(unit 1)
+					(variant
+						(name "5x5x5")
+						(dnp yes)
+					)
 				)
 			)
@@
 					(reference "C40")
 					(unit 1)
+					(variant
+						(name "5x5x5")
+						(dnp yes)
+					)
 				)
 			)
@@
 					(reference "U14")
 					(unit 1)
+					(variant
+						(name "5x5x5")
+						(dnp yes)
+					)
 				)
 			)
@@
 					(reference "C48")
 					(unit 1)
+					(variant
+						(name "5x5x5")
+						(dnp yes)
+					)
 				)
 			)
@@
 			)
 		)
-		(property "Value" "10R"
+		(property "Value" "100R"
 			(at 146.685 106.68 90)
 			(show_name no)
@@
 					(reference "Q3")
 					(unit 1)
+					(variant
+						(name "5x5x5")
+						(dnp yes)
+					)
 				)
 			)
@@
 			)
 		)
-		(property "Value" "10R"
+		(property "Value" "100R"
 			(at 146.685 50.8 90)
 			(show_name no)
@@
 					(reference "C29")
 					(unit 1)
+					(variant
+						(name "5x5x5")
+						(dnp yes)
+					)
 				)
 			)
@@
 					(reference "C19")
 					(unit 1)
+					(variant
+						(name "5x5x5")
+						(dnp yes)
+					)
 				)
 			)
@@
 					(reference "C18")
 					(unit 1)
+					(variant
+						(name "5x5x5")
+						(dnp yes)
+					)
 				)
 			)
@@
 					(reference "C30")
 					(unit 1)
+					(variant
+						(name "5x5x5")
+						(dnp yes)
+					)
 				)
 			)
@@
 					(reference "U3")
 					(unit 1)
+					(variant
+						(name "5x5x5")
+						(dnp yes)
+					)
 				)
 			)
@@
 					(reference "C43")
 					(unit 1)
+					(variant
+						(name "5x5x5")
+						(dnp yes)
+					)
 				)
 			)
@@
 					(reference "C21")
 					(unit 1)
+					(variant
+						(name "5x5x5")
+						(dnp yes)
+					)
 				)
 			)
@@
 					(reference "C22")
 					(unit 1)
+					(variant
+						(name "5x5x5")
+						(dnp yes)
+					)
 				)
 			)
@@
 			)
 		)
-		(property "Value" "10R"
+		(property "Value" "100R"
 			(at 69.215 107.315 90)
 			(show_name no)
@@
 					(reference "C31")
 					(unit 1)
+					(variant
+						(name "5x5x5")
+						(dnp yes)
+					)
 				)
 			)
@@
 					(reference "R46")
 					(unit 1)
+					(variant
+						(name "5x5x5")
+						(dnp yes)
+					)
 				)
 			)
@@
 			)
 		)
-		(property "Value" "10R"
+		(property "Value" "100R"
 			(at 302.26 49.53 90)
 			(show_name no)
@@
 					(reference "R35")
 					(unit 1)
+					(variant
+						(name "5x5x5")
+						(dnp yes)
+					)
 				)
 			)
@@
 					(reference "C20")
 					(unit 1)
+					(variant
+						(name "5x5x5")
+						(dnp yes)
+					)
 				)
 			)
@@
 					(reference "U7")
 					(unit 1)
+					(variant
+						(name "5x5x5")
+						(dnp yes)
+					)
 				)
 			)
@@
 			)
 		)
-		(property "Value" "10R"
+		(property "Value" "100R"
 			(at 69.215 51.435 90)
 			(show_name no)
@@
 					(reference "U10")
 					(unit 1)
+					(variant
+						(name "5x5x5")
+						(dnp yes)
+					)
 				)
 			)
@@
 					(reference "C42")
 					(unit 1)
+					(variant
+						(name "5x5x5")
+						(dnp yes)
+					)
 				)
 			)
@@
 					(reference "C41")
 					(unit 1)
+					(variant
+						(name "5x5x5")
+						(dnp yes)
+					)
 				)
 			)
@@
 			)
 		)
-		(property "Value" "10R"
+		(property "Value" "100R"
 			(at 224.79 50.165 90)
 			(show_name no)
@@
 					(reference "R36")
 					(unit 1)
+					(variant
+						(name "5x5x5")
+						(dnp yes)
+					)
 				)
 			)
@@
 					(reference "C39")
 					(unit 1)
+					(variant
+						(name "5x5x5")
+						(dnp yes)
+					)
 				)
 			)
@@
 					(reference "C38")
 					(unit 1)
+					(variant
+						(name "5x5x5")
+						(dnp yes)
+					)
 				)
 			)
@@
 			)
 		)
-		(property "Value" "10R"
+		(property "Value" "100R"
 			(at 146.685 162.56 90)
 			(show_name no)
@@
 					(reference "R43")
 					(unit 1)
+					(variant
+						(name "5x5x5")
+						(dnp yes)
+					)
 				)
 			)
@@
 					(reference "Q7")
 					(unit 1)
+					(variant
+						(name "5x5x5")
+						(dnp yes)
+					)
 				)
 			)
@@
 					(reference "Q10")
 					(unit 1)
+					(variant
+						(name "5x5x5")
+						(dnp yes)
+					)
 				)
 			)
@@
 					(reference "U4")
 					(unit 1)
+					(variant
+						(name "5x5x5")
+						(dnp yes)
+					)
 				)
 			)
@@
 			)
 		)
-		(property "Value" "10R"
+		(property "Value" "100R"
 			(at 69.215 163.195 90)
 			(show_name no)
@@
 					(reference "C17")
 					(unit 1)
+					(variant
+						(name "5x5x5")
+						(dnp yes)
+					)
 				)
 			)
@@
 					(reference "Q11")
 					(unit 1)
+					(variant
+						(name "5x5x5")
+						(dnp yes)
+					)
 				)
 			)
@@
 			)
 		)
-		(property "Value" "10R"
+		(property "Value" "100R"
 			(at 224.79 161.925 90)
 			(show_name no)
@@
 					(reference "R42")
 					(unit 1)
+					(variant
+						(name "5x5x5")
+						(dnp yes)
+					)
 				)
 			)
