File: SC_LED_CUBE_SLAVE_Board/SC_LED_CUBE_SLAVE_Board.kicad_sch (KiCad schematic)
At the start: 30 parts, among them CN1 XT30UPB-M, CN2 B03B-XASK-1-A(LF)(SN), CN3 B03B-XASK-1-A(LF)(SN), CN4 B03B-XASK-1-A(LF)(SN), CN5 B03B-XASK-1-A(LF)(SN), Q2 PMZ600UNEYL, Q3 PMZ600UNEYL, U2 STP16CPC26XTR, U3 STP16CPC26XTR

Commit message: Started the layout of the slave board.
Parts:
- added H1, H2, H3, H4: MountingHole_Pad, MountingHole:MountingHole_3.2mm_M3_Pad_Via, symbol Mechanical:MountingHole_Pad
- added R21, R22, R23, R24, R25, R26, R27, R28, R29, R30, R31, R32, R33, R34, R35, R36, R37, R38, R39, R40, R41, R42, R43, R44, R45: 1R, Resistor_SMD:R_0402_1005Metric_Pad0.72x0.64mm_HandSolder, symbol Device:R
Connections:
- net GND: now also H1.1, H2.1, H3.1, H4.1
- net O0: now also R45.2; no longer LC1.25 (LED25)
- net O1: now also R44.2; no longer LC1.24 (LED24)
- net O10: now also R35.2; no longer LC1.15 (LED15)
- net O11: now also R34.2; no longer LC1.14 (LED14)
- net O12: now also R33.2; no longer LC1.13 (LED13)
- net O13: now also R32.2; no longer LC1.12 (LED12)
- net O14: now also R31.2; no longer LC1.11 (LED11)
- net O15: now also R30.2; no longer LC1.10 (LED10)
- net O16: now also R29.2; no longer LC1.9 (LED9)
- net O17: now also R28.2; no longer LC1.8 (LED8)
- net O18: now also R27.2; no longer LC1.7 (LED7)
- net O19: now also R26.2; no longer LC1.6 (LED6)
- net O2: now also R43.2; no longer LC1.23 (LED23)
- net O20: now also R25.2; no longer LC1.5 (LED5)
- net O21: now also R24.2; no longer LC1.4 (LED4)
- net O22: now also R23.2; no longer LC1.3 (LED3)
- net O23: now also R22.2; no longer LC1.2 (LED2)
- net O24: now also R21.2; no longer LC1.1 (LED1)
- net O3: now also R42.2; no longer LC1.22 (LED22)
- net O4: now also R41.2; no longer LC1.21 (LED21)
- net O5: now also R40.2; no longer LC1.20 (LED20)
- net O6: now also R39.2; no longer LC1.19 (LED19)
- net O7: now also R38.2; no longer LC1.18 (LED18)
- net O8: now also R37.2; no longer LC1.17 (LED17)
- net O9: now also R36.2; no longer LC1.16 (LED16)
- new net: LC1.20 (LED20), R40.1
- new net: LC1.11 (LED11), R31.1
- new net: LC1.18 (LED18), R38.1
- new net: LC1.4 (LED4), R24.1
- new net: LC1.22 (LED22), R42.1
- new net: LC1.7 (LED7), R27.1
- new net: LC1.10 (LED10), R30.1
- new net: LC1.1 (LED1), R21.1
- new net: LC1.23 (LED23), R43.1
- new net: LC1.6 (LED6), R26.1
- new net: LC1.2 (LED2), R22.1
- new net: LC1.9 (LED9), R29.1
- new net: LC1.13 (LED13), R33.1
- new net: LC1.14 (LED14), R34.1
- new net: LC1.16 (LED16), R36.1
- new net: LC1.3 (LED3), R23.1
- new net: LC1.5 (LED5), R25.1
- new net: LC1.21 (LED21), R41.1
- new net: LC1.19 (LED19), R39.1
- new net: LC1.25 (LED25), R45.1
- new net: LC1.17 (LED17), R37.1
- new net: LC1.8 (LED8), R28.1
- new net: LC1.24 (LED24), R44.1
- new net: LC1.15 (LED15), R35.1
- new net: LC1.12 (LED12), R32.1

Commit message: Finished the layout 0 DRC errors.
Parts:
- added C44, C45, C46, C47, C48: 100uF, Capacitor_SMD:C_1206_3216Metric_Pad1.33x1.80mm_HandSolder, symbol Device:C
- added C49: 270uF, Capacitor_THT:CP_Radial_D6.3mm_P2.50mm, symbol Device:C_Polarized
- added R46, R47: 0R, Resistor_SMD:R_0402_1005Metric_Pad0.72x0.64mm_HandSolder, symbol Device:R
Connections:
- net GND: now also C44.2, C45.2, C46.2, C47.2, C48.2, C49.2
- net R_EXT: now also R47.2; no longer R6.1
- net VCC: now also C44.1, C45.1, C46.1, C47.1, C48.1, C49.1
- net at U2.23 (R-EXT): now also R46.1; no longer R1.1
- new net: R47.1, R6.1
- new net: R1.1, R46.2
Other:
- moved on the sheet: CN1

Commit message: Small mostly cosmetic changes, followed by the export of the gerber files for production.
Parts:
- renumbered C3 to C1, C42 to C10, C41 to C11, C40 to C12, C39 to C13, C38 to C14, C43 to C15, C49 to C16, C1 to C2, C4 to C3, C2 to C4, C48 to C5, C44 to C6, C45 to C7, C46 to C8, C47 to C9, CN4 to CN1, CN5 to CN3, CN3 to CN4, CN1 to CN5, FPC2 to FPC1, FPC1 to FPC2, Q2 to Q1, Q3 to Q2, R21 to R1, R26 to R10, R27 to R11, R28 to R12, R29 to R13, R30 to R14, R20 to R15, R2 to R16, R7 to R17, R5 to R18, R31 to R19, R22 to R2, R32 to R20, R33 to R21, R34 to R22, R35 to R23, R36 to R24, R37 to R25, R38 to R26, R39 to R27, R40 to R28, R16 to R29, R23 to R3, R41 to R30, R42 to R31, R43 to R32, R44 to R33, R45 to R34, R24 to R4, R25 to R5, R46 to R6, R47 to R7, R1 to R8, R6 to R9, U3 to U1
